Commit message: 2d cartographer node

File: gazebo/urdf/accessories/lidar3d.urdf.xacro (robot description, xacro)
@@ -1,5 +1,6 @@
 <?xml version="1.0"?>
 <robot xmlns:xacro="http://ros.org/wiki/xacro">
-  <xacro:macro name="add_lidar" params="parent_link">
+  <xacro:property name="M_PI" value="3.1415926535897931"/>
+  <xacro:macro name="add_lidar3D" params="parent_link">
     <joint name="laser_joint" type="fixed">
       <parent link="${parent_link}"/>
@@ -31,28 +32,49 @@
     </link>
     <gazebo reference="laser_frame">
-      <material>Gazebo/Blue</material>
+      <!-- <sensor type="ray" name="${name}-VLP16"> -->
       <sensor name="laser" type="ray">
-        <pose> 0 0 0 0 0 0 </pose>
+        <pose>0 0 0 0 0 0</pose>
         <visualize>true</visualize>
-        <update_rate>10</update_rate>
-        <!-- <update_rate>0.5</update_rate> -->
+        <update_rate>2</update_rate>
         <ray>
           <scan>
             <horizontal>
-              <samples>360</samples>
-              <min_angle>-3.14</min_angle>
-              <max_angle>3.14</max_angle>
+              <samples>440</samples>
+              <resolution>1</resolution>
+              <min_angle>-3.1415</min_angle>
+              <max_angle>3.1415</max_angle>
             </horizontal>
+            <vertical>
+              <samples>16</samples>
+              <resolution>1</resolution>
+              <min_angle>-${15.0*M_PI/180.0}</min_angle>
+              <max_angle>
+                ${15.0*M_PI/180.0}</max_angle>
+            </vertical>
           </scan>
           <range>
             <min>0.3</min>
-            <max>12</max>
+            <max>131</max>
+            <resolution>0.001</resolution>
           </range>
+          <noise>
+            <type>gaussian</type>
+            <mean>0.0</mean>
+            <stddev>0.0</stddev>
+          </noise>
         </ray>
+        <!-- <plugin name="laser_controller" filename="libgazebo_ros_velodyne_laser.so"> -->
+        <!-- <plugin name="laser_controller" filename="libgazebo_ros_block_laser.so">
+          <topicName>/scan</topicName>
+          <frameName>laser_scan</frameName>
+          <min_range>0.9</min_range>
+          <max_range>130</max_range>
+          <gaussianNoise>0.008</gaussianNoise>
+        </plugin> -->
         <plugin name="laser_controller" filename="libgazebo_ros_ray_sensor.so">
           <ros>
             <argument>~/out:=scan</argument>
           </ros>
-          <output_type>sensor_msgs/LaserScan</output_type>
+          <output_type>sensor_msgs/PointCloud2</output_type>
           <frame_name>laser_frame</frame_name>
         </plugin>

File: gazebo/urdf/husky_macro.urdf.xacro (robot description, xacro)
@@ -14,4 +14,5 @@
   <xacro:include filename="$(find trailbot_gazebo)/urdf/accessories/depth_camera.urdf.xacro"/>
   <xacro:include filename="$(find trailbot_gazebo)/urdf/accessories/lidar.urdf.xacro"/>
+  <!-- <xacro:include filename="$(find trailbot_gazebo)/urdf/accessories/lidar3d.urdf.xacro"/> -->
   <xacro:include filename="$(find trailbot_gazebo)/urdf/inertial_macros.xacro"/>
   <xacro:property name="M_PI" value="3.14159"/>
