Commit message: temp 3D work

File: gazebo/urdf/accessories/depth_camera.urdf.xacro (robot description, xacro)
@@ -18,5 +18,6 @@
       <parent link="camera_link"/>
       <child link="camera_link_optical"/>
-      <origin xyz="0 0 0" rpy="${-pi/2} 0 ${-pi/2}"/>
+      <!-- <origin xyz="0 0 0" rpy="${-pi/2} 0 ${-pi/2}"/> -->
+      <origin xyz="0 0 0" rpy="${-pi/2} 0 ${pi/2}"/>
     </joint>
     <link name="camera_link_optical"></link>

File: gazebo/urdf/accessories/lidar3D.urdf.xacro (robot description, xacro)
@@ -36,5 +36,5 @@
         <pose>0 0 0 0 0 0</pose>
         <visualize>true</visualize>
-        <update_rate>2</update_rate>
+        <update_rate>10</update_rate>
         <ray>
           <scan>

Commit message: working 3d costmap using pointcloud to laserscan

File: gazebo/urdf/accessories/depth_camera.urdf.xacro (robot description, xacro)
@@ -19,5 +19,6 @@
       <child link="camera_link_optical"/>
       <!-- <origin xyz="0 0 0" rpy="${-pi/2} 0 ${-pi/2}"/> -->
-      <origin xyz="0 0 0" rpy="${-pi/2} 0 ${pi/2}"/>
+      <!-- <origin xyz="0 0 0" rpy="${-pi/2} 0 ${pi/2}"/> -->
+      <origin xyz="0.33 0 0.90755" rpy="0 0 0"/>
     </joint>
     <link name="camera_link_optical"></link>

File: gazebo/urdf/accessories/lidar3D.urdf.xacro (robot description, xacro)
@@ -6,5 +6,6 @@
       <parent link="${parent_link}"/>
       <child link="laser_frame"/>
-      <origin xyz="0.0 -0.10 0.1" rpy="0 0 0"/>
+      <!-- <origin xyz="0.0 -0.10 0.1" rpy="0 0 0"/> -->
+      <origin xyz="0.236 0 1.0282" rpy="0 0 0"/>
     </joint>
     <link name="laser_frame">
@@ -35,5 +36,6 @@
       <sensor name="laser" type="ray">
         <pose>0 0 0 0 0 0</pose>
-        <visualize>true</visualize>
+        <!-- <visualize>true</visualize> -->
+        <visualize>false</visualize>
         <update_rate>10</update_rate>
         <ray>

File: gazebo/urdf/husky_macro.urdf.xacro (robot description, xacro)
@@ -109,7 +109,7 @@
       <child link="arch_top_link" />
     </joint>
-    <xacro:add_depth_camera parent_link="arch_top_link"/>
+    <xacro:add_depth_camera parent_link="base_link"/>
     <!-- <xacro:add_lidar parent_link="arch_top_link"/> -->
-    <xacro:add_lidar3D parent_link="arch_top_link"/>
+    <xacro:add_lidar3D parent_link="base_link"/>
     <ros2_control name="${prefix}husky_hardware" type="system">
       <hardware>

Commit message: changes to costmap size

File: gazebo/urdf/accessories/depth_camera.urdf.xacro (robot description, xacro)
@@ -5,5 +5,5 @@
       <parent link="${parent_link}"/>
       <child link="camera_link"/>
-      <origin xyz="0.0 0.1 0.015" rpy="0 0 0"/>
+      <origin xyz="0.33 0.1 0.921" rpy="0 0 0"/>
     </joint>
     <link name="camera_link">
