Commit message: velodyne joint

File: husky/husky_description/urdf/husky_macro.urdf.xacro (robot description, xacro)
@@ -82,5 +82,5 @@
     </link>
     <joint name="${prefix}velodyne_joint" type="fixed">
-      <origin xyz="0 0 0" rpy="0 0 0" />
+      <origin xyz="0.236 0 1.0282" rpy="0 0 0"/>
       <parent link="${prefix}base_link" />
       <child link="${prefix}velodyne" />

Commit message: necessary imu updates and rviz config

File: husky/husky_description/urdf/husky_macro.urdf.xacro (robot description, xacro)
@@ -91,4 +91,5 @@
     <joint name="${prefix}imu_joint" type="fixed">
       <origin xyz="$(optenv CPR_IMU_XYZ 0 0 0)" rpy="$(optenv CPR_IMU_RPY 0 0 0)" />
+      <!-- <origin xyz="0 -0.06 0.28" rpy="$(optenv CPR_IMU_RPY 0 0 0)" /> -->
       <parent link="${prefix}base_link" />
       <child link="${prefix}imu_link" />

Commit message: fixing the gps frame

File: husky/husky_description/urdf/husky_macro.urdf.xacro (robot description, xacro)
@@ -94,9 +94,16 @@
       <child link="${prefix}imu_link" />
     </joint>
-    <!-- GPS Link-->
+    <!-- GPS Link from base-->
+    <!-- Was 43cm back (x) from lidar, 20cm right (y) from lidar, and 17cm (z) higher-->
     <!-- Can be modified with environment variables in /etc/ros/setup.bash -->
-    <link name="${prefix}gps_link"/>
+    <link name="${prefix}gps_link">
+      <inertial>
+        <mass value="5.0" />
+        <origin xyz="-0.00065 -0.035 0.042" />
+        <inertia ixx="0.6022" ixy="-0.02364" ixz="-0.1197" iyy="1.7386" iyz="-0.001544" izz="2.0296" />
+      </inertial>
+    </link>
     <joint name="${prefix}gps_joint" type="fixed">
-      <origin xyz="$(optenv CPR_GPS_XYZ 0 0 0)" rpy="$(optenv CPR_GPS_RPY 0 0 0)" />
+      <origin xyz="-0.194 -0.20 1.20" rpy="0 0 0" />
       <parent link="${prefix}base_link" />
       <child link="${prefix}gps_link" />

Commit message: changes needed but issue with pcl2lserscan

File: husky/husky_description/urdf/husky_macro.urdf.xacro (robot description, xacro)
@@ -97,5 +97,5 @@
     <!-- Was 43cm back (x) from lidar, 20cm right (y) from lidar, and 17cm (z) higher-->
     <!-- Can be modified with environment variables in /etc/ros/setup.bash -->
-    <link name="${prefix}gps_link">
+    <link name="${prefix}gps">
       <inertial>
         <mass value="5.0" />
@@ -107,5 +107,5 @@
       <origin xyz="-0.194 -0.20 1.20" rpy="0 0 0" />
       <parent link="${prefix}base_link" />
-      <child link="${prefix}gps_link" />
+      <child link="${prefix}gps" />
     </joint>
     <!-- Husky wheel macros -->

Commit message: what to do if you want to use the gps

File: husky/husky_description/urdf/husky_macro.urdf.xacro (robot description, xacro)
@@ -96,9 +96,15 @@
     <!-- GPS Link-->
     <!-- Can be modified with environment variables in /etc/ros/setup.bash -->
-    <link name="${prefix}gps_link"/>
+    <link name="${prefix}gps">
+      <inertial>
+        <mass value="5.0" />
+        <origin xyz="-0.00065 -0.035 0.042" />
+        <inertia ixx="0.6022" ixy="-0.02364" ixz="-0.1197" iyy="1.7386" iyz="-0.001544" izz="2.0296" />
+      </inertial>
+    </link>
     <joint name="${prefix}gps_joint" type="fixed">
-      <origin xyz="$(optenv CPR_GPS_XYZ 0 0 0)" rpy="$(optenv CPR_GPS_RPY 0 0 0)" />
-      <parent link="${prefix}base_link" />
-      <child link="${prefix}gps_link" />
+      <origin xyz="-0.194 -0.20 1.10" rpy="0 0 0" />
+      <parent link="${prefix}base_link" />
+      <child link="${prefix}gps" />
     </joint>
     <!-- Husky wheel macros -->

Commit message: OS0-64 Lidar
added ros-drivers
cartographer unstable

File: husky/husky_description/urdf/husky_macro.urdf.xacro (robot description, xacro)
@@ -74,5 +74,5 @@
       <child link="${prefix}inertial_link" />
     </joint>
-    <link name="${prefix}velodyne">
+     <link name="${prefix}os_sensor">
       <inertial>
         <mass value="46.034" />
@@ -81,9 +81,21 @@
       </inertial>
     </link>
+    <joint name="${prefix}os_sensor_joint" type="fixed">
+      <origin xyz="0.236 0 1.0282" rpy="0 0 0"/>
+      <parent link="${prefix}base_link" />
+      <child link="${prefix}os_sensor" />
+    </joint>
+    <!-- <link name="${prefix}velodyne">
+      <inertial>
+        <mass value="46.034" />
+        <origin xyz="-0.00065 -0.085 0.062" />
+        <inertia ixx="0.6022" ixy="-0.02364" ixz="-0.1197" iyy="1.7386" iyz="-0.001544" izz="2.0296" />
+      </inertial>
+    </link>
     <joint name="${prefix}velodyne_joint" type="fixed">
       <origin xyz="0.236 0 1.0282" rpy="0 0 0"/>
       <parent link="${prefix}base_link" />
       <child link="${prefix}velodyne" />
-    </joint>
+    </joint> -->
     <!-- IMU Link-->
     <!-- Can be modified with environment variables in /etc/ros/setup.bash -->

Commit message: ouster-stable
IMU, LiDAR, carto, nav2 - SAT
carto, nav2 - not tuned
LiDAR urdf link corrected

File: husky/husky_description/urdf/husky_macro.urdf.xacro (robot description, xacro)
@@ -82,5 +82,5 @@
     </link>
     <joint name="${prefix}os_sensor_joint" type="fixed">
-      <origin xyz="0.236 0 1.0282" rpy="0 0 0"/>
+      <origin xyz="0.236 0 1.0282" rpy="0 0 ${M_PI/2}"/>
       <parent link="${prefix}base_link" />
       <child link="${prefix}os_sensor" />

Commit message: ouster imu setup
changed topics/frames to use ouster imu data
removed external imu_link
tuned cartogrpher (based on indoor-feb16 bag)

File: husky/husky_description/urdf/husky_macro.urdf.xacro (robot description, xacro)
@@ -98,12 +98,13 @@
       <child link="${prefix}velodyne" />
     </joint> -->
+    <!-- Suppressed ext. IMU, Internal IMU in OUSTER LiDAR system is being used, check TF tree and ouster/imu topic-->
     <!-- IMU Link-->
     <!-- Can be modified with environment variables in /etc/ros/setup.bash -->
-    <link name="${prefix}imu_link"/>
+    <!-- <link name="${prefix}imu_link"/>
     <joint name="${prefix}imu_joint" type="fixed">
       <origin xyz="$(optenv CPR_IMU_XYZ 0 0 0)" rpy="$(optenv CPR_IMU_RPY 0 0 0)" />
       <parent link="${prefix}base_link" />
       <child link="${prefix}imu_link" />
-    </joint>
+    </joint> -->
     <!-- GPS Link-->
     <!-- Can be modified with environment variables in /etc/ros/setup.bash -->

Commit message: Ouster Lidar  (#58)
* OS0-64 Lidar

added ros-drivers
cartographer unstable

* 2D Cartographer Fix

* ouster-carto3D

all nodes sat
carto params needs tuning

* ouster-stable

IMU, LiDAR, carto, nav2 - SAT
carto, nav2 - not tuned
LiDAR urdf link corrected

* ouster imu setup

changed topics/frames to use ouster imu data
removed external imu_link
tuned cartogrpher (based on indoor-feb16 bag)

* nav2 params update

-ouster launch is renamed to trailbot bringup (includes driving and other hardware initialization)

* param updates

-changed max_raytrace_range
-changed local costmap update frequency
-corrected lidar subscription topic in human detection node

---------

Co-authored-by: trailbot <nic.koenig37@gmail.com>

File: husky/husky_description/urdf/husky_macro.urdf.xacro (robot description, xacro)
@@ -74,5 +74,5 @@
       <child link="${prefix}inertial_link" />
     </joint>
-    <link name="${prefix}velodyne">
+     <link name="${prefix}os_sensor">
       <inertial>
         <mass value="46.034" />
@@ -81,17 +81,30 @@
       </inertial>
     </link>
+    <joint name="${prefix}os_sensor_joint" type="fixed">
+      <origin xyz="0.236 0 1.0282" rpy="0 0 ${M_PI/2}"/>
+      <parent link="${prefix}base_link" />
+      <child link="${prefix}os_sensor" />
+    </joint>
+    <!-- <link name="${prefix}velodyne">
+      <inertial>
+        <mass value="46.034" />
+        <origin xyz="-0.00065 -0.085 0.062" />
+        <inertia ixx="0.6022" ixy="-0.02364" ixz="-0.1197" iyy="1.7386" iyz="-0.001544" izz="2.0296" />
+      </inertial>
+    </link>
     <joint name="${prefix}velodyne_joint" type="fixed">
       <origin xyz="0.236 0 1.0282" rpy="0 0 0"/>
       <parent link="${prefix}base_link" />
       <child link="${prefix}velodyne" />
-    </joint>
+    </joint> -->
+    <!-- Suppressed ext. IMU, Internal IMU in OUSTER LiDAR system is being used, check TF tree and ouster/imu topic-->
     <!-- IMU Link-->
     <!-- Can be modified with environment variables in /etc/ros/setup.bash -->
-    <link name="${prefix}imu_link"/>
+    <!-- <link name="${prefix}imu_link"/>
     <joint name="${prefix}imu_joint" type="fixed">
       <origin xyz="$(optenv CPR_IMU_XYZ 0 0 0)" rpy="$(optenv CPR_IMU_RPY 0 0 0)" />
       <parent link="${prefix}base_link" />
       <child link="${prefix}imu_link" />
-    </joint>
+    </joint> -->
     <!-- GPS Link-->
     <!-- Can be modified with environment variables in /etc/ros/setup.bash -->
